File: mux-shield-pcb/mux-shield-pcb.brd (EAGLE design)
At the start: 68.6 x 53.3 mm, 12 parts, among them X1 BN35N61, X2 BN35N61, X3 BU-SMB-V, X4 BU-SMB-V, X5 BU-SMA-V

Commit message: Update PCB connecting button to ground rather than 5V
Connections:
- net +5V: no longer S1.1, S1.2
- net GND: now also S1.1, S1.2
Routing:
- net +5V: track 75.3 -> 0.00 mm
- net GND: track 144.5 -> 168.6 mm, vias 0 -> 1
- net N$8: track 45.3 -> 58.9 mm
- net N$9: track 48.9 -> 57.7 mm
- net N$5: track 47.0 -> 45.4 mm
- net N$6: track 43.1 -> 41.6 mm
Other:
- board text added: "v1.1"
